File: pcb/seedjoy_testboard.kicad_pcb (KiCad board)
At the start: 2 copper layers, 130 x 75 mm, 27 parts, among them J1 XIAO_L, J2 XIAO_R, J3 THUMBSTICK, J4 X_SEL, J5 Y_SEL, J6 STICK_BTN_EN, J7 SR_CHAIN_IN, J8 X_SRC, J9 Y_SRC, SW1 BTN1, SW2 BTN2, SW3 BTN3, SW4 BTN4, SW5 BTN5, SW6 BTN6, SW7 BTN7, SW8 BTN8, SW9 GPIO/MODE, U1 74HC165, U2 RKJXV1224005

Commit message: fix: audit firmware, configurator and test board against real hardware
Firmware
- Axes use a ratiometric ADC reference (AR_VDD4): 0..4095 == 0..VDD, so a
  3.3 V pot centres at ~2048. AR_DEFAULT (3.6 V internal) capped the stick
  at ~3750 with centre ~1877, outside the default calibration.
- Hold VBAT_ENABLE (P0.14) LOW from boot and never release it; a floating
  P0.14 lets P0.31 rise toward raw VBAT, above the nRF52840 3.6 V abs max.
- New serial commands stream_axes / stop_axes (20 Hz raw + processed).

Configurator
- Calibration over USB Serial was showing SIMULATED axis movement: the
  firmware never sent axis data over serial, serial.js lacked isConnected(),
  and onAxisData was only wired to the BLE client. Stream axes on the
  calibration tab, wire both transports, and never fall back to simulated
  values (or capture them for min/center/max) while a device is connected.

Test board
- Silkscreen: HID 1-8 requires "Number of chips = 1" (firmware default 7
  would put the board's buttons at HID 49-56). Gerbers regenerated.
- pcb/README.md: bring-up checklist (pre-order stick measurement, bare
  board checks, assembly order, first power-up, configuration, jumpers).

Verified: firmware + FFB build compile, host tests pass; configurator's real
write_config payload parsed by the firmware's real JSON code on host and
round-tripped through read_config; PCB pad nets extracted from the board
match the firmware pin map; XIAO pinout/orientation checked against
Seeed's official KiCad symbol and footprint; bootloader DFU pins
(P0.18 + P0.03 together) confirmed not triggerable by the board. DRC 0
errors / 0 unconnected.

Co-Authored-By: Claude Opus 5.5 <noreply@anthropic.com>
Other:
- board text added: "BTN1-8 = HID 1-8 (configurator: Number of chips = 1)"
- board text removed: "BTN1 ... BTN8 (HID 1-8)"
Changed lines of the file:
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@@
 		)
 	)
-	(gr_text "BTN1 ... BTN8 (HID 1-8)"
+	(gr_text "BTN1-8 = HID 1-8 (configurator: Number of chips = 1)"
 		(at 150 165 0)
 		(layer "F.SilkS")
